File: Headend.sch (EAGLE design)
At the start: 56 parts, among them IC1 317EMP, Q1 12.288Mhz, SW1 SPST_TACT-KMR2, U1 TXS0102

Commit message: Update board design
Connections:
- removed net N$12: COMMS_CPU.GPIO15, R8.1
- removed net N$6: COMMS_CPU.RESET, R9.1, SW1.P, SW1.P1
- new net TEENSYCS: COMMS_CPU.GPIO15, R8.2, UI_CPU.10/TX2/PWM
- new net WATCHDOG: COMMS_CPU.RESET, R9.1, SW1.P, SW1.P1, UI_CPU.2
- net +3V3: no longer R8.2
- net GND: now also R8.1
Other:
- moved on the sheet: R10, R8, R9, SW1, TOUCH

Commit message: Update board with further tweaks
Parts:
- removed SW1: SPST_TACT-KMR2, adafruit:SPST_TACT-KMR2
- added C22, C23: 10uF, adafruit:C-USC0402
- added PGM_SW: SPST_TACT-KMR2, adafruit:SPST_TACT-KMR2
- C1, C2: value 8uF -> 10uF
- C13, C14: value 33pF -> 10pF
Connections:
- net +3V3: now also C22.1, C23.1
- net GND: now also C22.2, C23.2, PGM_SW.S, PGM_SW.S1; no longer SW1.S, SW1.S1
- net WATCHDOG: now also RESET_SW.P, RESET_SW.P1; no longer SW1.P, SW1.P1
- net XDCS: now also PGM_SW.P, PGM_SW.P1; no longer RESET_SW.P, RESET_SW.P1
Other:
- moved on the sheet: R16, R5, RESET_SW

Commit message: Update design, clean up spurious resistor between 3v3 and Gnd, clean up some routing
Parts:
- removed R14: 10k, adafruit:R-US_R0402
Connections:
- net +3V3: no longer R14.1
- net GND: no longer R14.2
Changed lines of the file:
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@@
 <grid distance="0.1" unitdist="inch" unit="inch" style="lines" multiple="1" display="no" altdistance="0.01" altunitdist="inch" altunit="inch"/>
 <layers>
-<layer number="1" name="Top" color="4" fill="1" visible="yes" active="no"/>
-<layer number="16" name="Bottom" color="1" fill="1" visible="yes" active="no"/>
-<layer number="17" name="Pads" color="2" fill="1" visible="yes" active="no"/>
-<layer number="18" name="Vias" color="2" fill="1" visible="yes" active="no"/>
-<layer number="19" name="Unrouted" color="6" fill="1" visible="yes" active="no"/>
-<layer number="20" name="Dimension" color="15" fill="1" visible="yes" active="no"/>
-<layer number="21" name="tPlace" color="7" fill="1" visible="yes" active="no"/>
-<layer number="22" name="bPlace" color="7" fill="1" visible="yes" active="no"/>
-<layer number="23" name="tOrigins" color="15" fill="1" visible="yes" active="no"/>
-<layer number="24" name="bOrigins" color="15" fill="1" visible="yes" active="no"/>
-<layer number="25" name="tNames" color="7" fill="1" visible="yes" active="no"/>
-<layer number="26" name="bNames" color="7" fill="1" visible="yes" active="no"/>
-<layer number="27" name="tValues" color="7" fill="1" visible="yes" active="no"/>
-<layer number="28" name="bValues" color="7" fill="1" visible="yes" active="no"/>
+<layer number="1" name="Top" color="4" fill="1" visible="no" active="no"/>
+<layer number="16" name="Bottom" color="1" fill="1" visible="no" active="no"/>
+<layer number="17" name="Pads" color="2" fill="1" visible="no" active="no"/>
+<layer number="18" name="Vias" color="2" fill="1" visible="no" active="no"/>
+<layer number="19" name="Unrouted" color="6" fill="1" visible="no" active="no"/>
+<layer number="20" name="Dimension" color="15" fill="1" visible="no" active="no"/>
+<layer number="21" name="tPlace" color="7" fill="1" visible="no" active="no"/>
+<layer number="22" name="bPlace" color="7" fill="1" visible="no" active="no"/>
+<layer number="23" name="tOrigins" color="15" fill="1" visible="no" active="no"/>
+<layer number="24" name="bOrigins" color="15" fill="1" visible="no" active="no"/>
+<layer number="25" name="tNames" color="7" fill="1" visible="no" active="no"/>
+<layer number="26" name="bNames" color="7" fill="1" visible="no" active="no"/>
+<layer number="27" name="tValues" color="7" fill="1" visible="no" active="no"/>
+<layer number="28" name="bValues" color="7" fill="1" visible="no" active="no"/>
 <layer number="29" name="tStop" color="7" fill="3" visible="no" active="no"/>
 <layer number="30" name="bStop" color="7" fill="6" visible="no" active="no"/>
@@
 <layer number="35" name="tGlue" color="7" fill="4" visible="no" active="no"/>
 <layer number="36" name="bGlue" color="7" fill="5" visible="no" active="no"/>
-<layer number="37" name="tTest" color="7" fill="1" visible="yes" active="no"/>
-<layer number="38" name="bTest" color="7" fill="1" visible="yes" active="no"/>
+<layer number="37" name="tTest" color="7" fill="1" visible="no" active="no"/>
+<layer number="38" name="bTest" color="7" fill="1" visible="no" active="no"/>
 <layer number="39" name="tKeepout" color="4" fill="11" visible="no" active="no"/>
 <layer number="40" name="bKeepout" color="1" fill="11" visible="no" active="no"/>
@@
 <layer number="44" name="Drills" color="7" fill="1" visible="no" active="no"/>
 <layer number="45" name="Holes" color="7" fill="1" visible="no" active="no"/>
-<layer number="46" name="Milling" color="3" fill="1" visible="yes" active="no"/>
-<layer number="47" name="Measures" color="7" fill="1" visible="yes" active="no"/>
-<layer number="48" name="Document" color="7" fill="1" visible="yes" active="no"/>
-<layer number="49" name="Reference" color="7" fill="1" visible="yes" active="no"/>
-<layer number="50" name="dxf" color="7" fill="1" visible="yes" active="no"/>
-<layer number="51" name="tDocu" color="7" fill="1" visible="yes" active="no"/>
-<layer number="52" name="bDocu" color="7" fill="1" visible="yes" active="no"/>
-<layer number="53" name="tGND_GNDA" color="7" fill="9" visible="yes" active="no"/>
-<layer number="54" name="bGND_GNDA" color="1" fill="9" visible="yes" active="no"/>
-<layer number="56" name="wert" color="7" fill="1" visible="yes" active="no"/>
+<layer number="46" name="Milling" color="3" fill="1" visible="no" active="no"/>
+<layer number="47" name="Measures" color="7" fill="1" visible="no" active="no"/>
+<layer number="48" name="Document" color="7" fill="1" visible="no" active="no"/>
+<layer number="49" name="Reference" color="7" fill="1" visible="no" active="no"/>
+<layer number="50" name="dxf" color="7" fill="1" visible="no" active="no"/>
+<layer number="51" name="tDocu" color="7" fill="1" visible="no" active="no"/>
+<layer number="52" name="bDocu" color="7" fill="1" visible="no" active="no"/>
+<layer number="53" name="tGND_GNDA" color="7" fill="9" visible="no" active="no"/>
+<layer number="54" name="bGND_GNDA" color="1" fill="9" visible="no" active="no"/>
+<layer number="56" name="wert" color="7" fill="1" visible="no" active="no"/>
 <layer number="91" name="Nets" color="2" fill="1" visible="yes" active="yes"/>
 <layer number="92" name="Busses" color="1" fill="1" visible="yes" active="yes"/>
@@
 <part name="ESP_FTDI" library="con-lstb" deviceset="MA04-1" device=""/>
 <part name="+3V11" library="supply1" deviceset="+3V3" device=""/>
-<part name="R14" library="adafruit" deviceset="R-US_" device="R0402" value="10k"/>
 <part name="STANDOFF1" library="SparkFun-Electromechanical" deviceset="STAND-OFF" device=""/>
 <part name="STANDOFF2" library="SparkFun-Electromechanical" deviceset="STAND-OFF" device=""/>
@@
 <instance part="ESP_FTDI" gate="1" x="134.62" y="152.4" rot="R180"/>
 <instance part="+3V11" gate="G$1" x="99.06" y="180.34"/>
-<instance part="R14" gate="G$1" x="78.74" y="144.78" rot="R270"/>
 <instance part="STANDOFF1" gate="G$1" x="378.46" y="38.1"/>
 <instance part="STANDOFF2" gate="G$1" x="378.46" y="33.02"/>
@@
 <junction x="101.6" y="139.7"/>
 <pinref part="ESP_FTDI" gate="1" pin="4"/>
-<pinref part="R14" gate="G$1" pin="2"/>
-<wire x1="78.74" y1="139.7" x2="101.6" y2="139.7" width="0.1524" layer="91"/>
+<wire x1="71.12" y1="139.7" x2="101.6" y2="139.7" width="0.1524" layer="91"/>
 <pinref part="C23" gate="G$1" pin="2"/>
 <wire x1="71.12" y1="162.56" x2="71.12" y2="139.7" width="0.1524" layer="91"/>
-<wire x1="71.12" y1="139.7" x2="78.74" y2="139.7" width="0.1524" layer="91"/>
-<junction x="78.74" y="139.7"/>
 </segment>
 <segment>
@@
 <wire x1="99.06" y1="170.18" x2="99.06" y2="172.72" width="0.1524" layer="91"/>
 <wire x1="99.06" y1="172.72" x2="99.06" y2="177.8" width="0.1524" layer="91"/>
-<wire x1="78.74" y1="149.86" x2="78.74" y2="172.72" width="0.1524" layer="91"/>
 <junction x="99.06" y="172.72"/>
-<pinref part="R14" gate="G$1" pin="1"/>
 <pinref part="R15" gate="G$1" pin="1"/>
-<wire x1="78.74" y1="172.72" x2="83.82" y2="172.72" width="0.1524" layer="91"/>
 <wire x1="83.82" y1="172.72" x2="99.06" y2="172.72" width="0.1524" layer="91"/>
 <wire x1="83.82" y1="170.18" x2="83.82" y2="172.72" width="0.1524" layer="91"/>
 <junction x="83.82" y="172.72"/>
 <pinref part="C23" gate="G$1" pin="1"/>
-<wire x1="78.74" y1="172.72" x2="71.12" y2="172.72" width="0.1524" layer="91"/>
+<wire x1="83.82" y1="172.72" x2="71.12" y2="172.72" width="0.1524" layer="91"/>
 <wire x1="71.12" y1="172.72" x2="71.12" y2="170.18" width="0.1524" layer="91"/>
-<junction x="78.74" y="172.72"/>
-</segment>
-<segment>
+</segment>
+<segment>

Commit message: Updated with more reddit feedback
Parts:
- removed IC1: 317EMP, linear:317EMP
- removed R1: 240, adafruit:R-US_R0603
- removed R2: 106, adafruit:R-US_R0603
- added C24: 1uF, adafruit:C-USC0402
- added C25: 4.7uF, adafruit:CPOL-USA
- added SJ1: (no value), jumper:SJ
- added U2: AP7313, CustomParts:AP7313
- AUDIO_CPU: value VS1033 -> VS1063
- C20: value 0.1uF -> 1uF
Connections:
- removed net N$5: IC1.ADJ, R1.2, R2.1
- new net AGND: AUDIO_CPU.AGND1, AUDIO_CPU.AGND2, AUDIO_CPU.AGND3, AUDIO_CPU.AGND4, AUDIO_OUT.1, C15.2, C16.2, SJ1.2
- net +3V3: now also C24.1, C25.+; no longer C20.1, IC1.VI
- net +5V: now also C20.1, U2.IN
- net 1.8V: now also U2.OUT; no longer IC1.VO, R1.1
- net GND: now also C24.2, C25.-, SJ1.1, U2.GND; no longer AUDIO_CPU.AGND1, AUDIO_CPU.AGND2, AUDIO_CPU.AGND3, AUDIO_CPU.AGND4, AUDIO_OUT.1, C15.2, C16.2, R2.2
- net WATCHDOG: no longer RESET_SW.P
- net XDCS: no longer PGM_SW.P
Other:
- moved on the sheet: C19, C20
